File: pcb/demo.kicad_sch (KiCad schematic)
At the start: 18 parts, among them J1 Conn_01x01_Pin, J2 Conn_01x01_Pin, Q1 BC547, Q2 BC547

Commit message: Add vendor
Parts:
- C1, C2: Vendor (none) -> HTL; VendorId (none) -> 100354
- D1, D2: Vendor (none) -> HTL; VendorId (none) -> 100445, 100444
- H1, H2: Vendor (none) -> HTL; VendorId (none) -> 101017, 101382
- J1, J2: Vendor (none) -> HTL; VendorId (none) -> 101521
- Q1, Q2: Vendor (none) -> HTL; VendorId (none) -> 100215
- R1, R2: Vendor (none) -> HTL; VendorId (none) -> 102800
- R3, R4: Vendor (none) -> HTL; VendorId (none) -> 102812
Changed lines of the file:
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@@
+      (effects (font (size 1.27 1.27)) hide)
+    )
+    (property "Vendor" "HTL" (at 177.8 95.25 0)
+      (effects (font (size 1.27 1.27)) hide)
+    )
+    (property "VendorId" "102800" (at 177.8 95.25 0)
       (effects (font (size 1.27 1.27)) hide)
     )
@@
       (effects (font (size 1.27 1.27)) hide)
     )
+    (property "Vendor" "" (at 38.1 165.1 0)
+      (effects (font (size 1.27 1.27)) hide)
+    )
+    (property "VendorId" "" (at 38.1 165.1 0)
+      (effects (font (size 1.27 1.27)) hide)
+    )
     (instances
       (project "demo"
@@
       (effects (font (size 1.27 1.27)) hide)
     )
+    (property "Vendor" "" (at 50.8 165.1 0)
+      (effects (font (size 1.27 1.27)) hide)
+    )
+    (property "VendorId" "" (at 50.8 165.1 0)
+      (effects (font (size 1.27 1.27)) hide)
+    )
     (instances
       (project "demo"
@@
     )
     (property "Datasheet" "~" (at 158.75 88.9 0)
+      (effects (font (size 1.27 1.27)) hide)
+    )
+    (property "Vendor" "HTL" (at 158.75 88.9 0)
+      (effects (font (size 1.27 1.27)) hide)
+    )
+    (property "VendorId" "102812" (at 158.75 88.9 0)
       (effects (font (size 1.27 1.27)) hide)
     )
@@
       (effects (font (size 1.27 1.27)) hide)
     )
+    (property "Vendor" "HTL" (at 129.54 114.3 0)
+      (effects (font (size 1.27 1.27)) hide)
+    )
+    (property "VendorId" "100215" (at 129.54 114.3 0)
+      (effects (font (size 1.27 1.27)) hide)
+    )
     (pin "1")
     (pin "2")
@@
       (effects (font (size 1.27 1.27)) hide)
     )
+    (property "Vendor" "HTL" (at 177.8 82.55 0)
+      (effects (font (size 1.27 1.27)) hide)
+    )
+    (property "VendorId" "100445, 100444" (at 177.8 82.55 0)
+      (effects (font (size 1.27 1.27)) hide)
+    )
     (pin "1")
     (pin "2")
@@
       (effects (font (size 1.27 1.27)) hide)
     )
+    (property "Vendor" "HTL" (at 165.1 104.14 0)
+      (effects (font (size 1.27 1.27)) hide)
+    )
+    (property "VendorId" "100354" (at 165.1 104.14 0)
+      (effects (font (size 1.27 1.27)) hide)
+    )
     (pin "1")
     (pin "2")
@@
       (effects (font (size 1.27 1.27)) hide)
     )
+    (property "Vendor" "HTL" (at 109.22 121.92 0)
+      (effects (font (size 1.27 1.27)) hide)
+    )
+    (property "VendorId" "101521" (at 109.22 121.92 0)
+      (effects (font (size 1.27 1.27)) hide)
+    )
     (pin "1")
     (instances
@@
     )
     (property "Datasheet" "~" (at 146.05 88.9 0)
+      (effects (font (size 1.27 1.27)) hide)
+    )
+    (property "Vendor" "HTL" (at 146.05 88.9 0)
+      (effects (font (size 1.27 1.27)) hide)
+    )
+    (property "VendorId" "102812" (at 146.05 88.9 0)
       (effects (font (size 1.27 1.27)) hide)
     )
@@
       (effects (font (size 1.27 1.27)) hide)
     )
+    (property "Vendor" "HTL" (at 175.26 114.3 0)
+      (effects (font (size 1.27 1.27)) hide)
+    )
+    (property "VendorId" "100215" (at 175.26 114.3 0)
+      (effects (font (size 1.27 1.27)) hide)
+    )
     (pin "1")
     (pin "2")
@@
     )
     (property "Datasheet" "~" (at 139.7 104.14 0)
+      (effects (font (size 1.27 1.27)) hide)
+    )
+    (property "Vendor" "HTL" (at 139.7 104.14 0)
+      (effects (font (size 1.27 1.27)) hide)
+    )
+    (property "VendorId" "100354" (at 139.7 104.14 0)
       (effects (font (size 1.27 1.27)) hide)
     )
@@
       (effects (font (size 1.27 1.27)) hide)
     )
+    (property "Vendor" "HTL" (at 114.3 166.37 0)
+      (effects (font (size 1.27 1.27)) hide)
+    )
+    (property "VendorId" "101017, 101382" (at 114.3 166.37 0)
+      (effects (font (size 1.27 1.27)) hide)
+    )
     (pin "1")
     (instances
@@
       (effects (font (size 1.27 1.27)) hide)
     )
+    (property "Vendor" "HTL" (at 101.6 166.37 0)
+      (effects (font (size 1.27 1.27)) hide)
+    )
+    (property "VendorId" "101017, 101382" (at 101.6 166.37 0)
+      (effects (font (size 1.27 1.27)) hide)
+    )
     (pin "1")
     (instances
@@
     )
     (property "Datasheet" "~" (at 109.22 76.2 0)
+      (effects (font (size 1.27 1.27)) hide)
+    )
+    (property "Vendor" "HTL" (at 109.22 76.2 0)
+      (effects (font (size 1.27 1.27)) hide)
+    )
+    (property "VendorId" "101521" (at 109.22 76.2 0)
       (effects (font (size 1.27 1.27)) hide)
     )
@@
       (effects (font (size 1.27 1.27)) hide)
     )
+    (property "Vendor" "HTL" (at 127 82.55 0)
+      (effects (font (size 1.27 1.27)) hide)
+    )
+    (property "VendorId" "100445, 100444" (at 127 82.55 0)
+      (effects (font (size 1.27 1.27)) hide)
+    )
     (pin "1")
     (pin "2")
@@
       (effects (font (size 1.27 1.27)) hide)
     )
+    (property "Vendor" "" (at 76.2 165.1 0)
+      (effects (font (size 1.27 1.27)) hide)
+    )
+    (property "VendorId" "" (at 76.2 165.1 0)
+      (effects (font (size 1.27 1.27)) hide)
+    )
     (instances
       (project "demo"
@@
       (effects (font (size 1.27 1.27)) hide)
     )
+    (property "Vendor" "" (at 63.5 165.1 0)
+      (effects (font (size 1.27 1.27)) hide)
+    )
+    (property "VendorId" "" (at 63.5 165.1 0)
+      (effects (font (size 1.27 1.27)) hide)
+    )
     (instances
       (project "demo"
@@
       (effects (font (size 1.27 1.27)) hide)
     )
+    (property "Vendor" "HTL" (at 127 95.25 0)
+      (effects (font (size 1.27 1.27)) hide)
+    )
+    (property "VendorId" "102800" (at 127 95.25 0)
+      (effects (font (size 1.27 1.27)) hide)
+    )
